File: badUSB/badUSB.kicad_sch (KiCad schematic)
At the start: 6 parts, among them J1 USB_A, SW1 SW_Push, U1 CH552G

Commit message: footprints added
Parts:
- C1, C2: footprint (none) -> Capacitor_SMD:C_0603_1608Metric
- R1: footprint (none) -> Resistor_SMD:R_0603_1608Metric
- U1: footprint (none) -> Package_SO:SOIC-16_3.9x9.9mm_P1.27mm
Changed lines of the file:
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@@
 			)
 		)
-		(property "Footprint" ""
+		(property "Footprint" "Capacitor_SMD:C_0603_1608Metric"
 			(at 125.73 43.4848 0)
 			(hide yes)
@@
 			)
 		)
-		(property "Footprint" ""
+		(property "Footprint" "Resistor_SMD:R_0603_1608Metric"
 			(at 93.472 48.26 90)
 			(hide yes)
@@
 			)
 		)
-		(property "Footprint" ""
+		(property "Footprint" "Package_SO:SOIC-16_3.9x9.9mm_P1.27mm"
 			(at 125.73 60.96 0)
 			(hide yes)
@@
 	)
 	(symbol
+		(lib_name "C_1")
 		(lib_id "Device:C")
 		(at 133.35 44.45 90)
@@
 			)
 		)
-		(property "Footprint" ""
+		(property "Footprint" "Capacitor_SMD:C_0603_1608Metric"
 			(at 137.16 43.4848 0)
 			(hide yes)

Commit message: pcb work
Parts:
- added D1, D2, D3: LED, LED_SMD:LED_0805_2012Metric, symbol Device:LED
- added R2, R3, R4: 330R, Resistor_SMD:R_0603_1608Metric, symbol Device:R
- added SW2: SW_Push, Button_Switch_SMD:SW_Tactile_SPST_NO_Straight_CK_PTS636Sx25SMTRLFS, symbol Switch:SW_Push
- SW1: footprint Button_Switch_THT:SW_PUSH_6mm_H5mm -> Button_Switch_SMD:SW_Tactile_SPST_NO_Straight_CK_PTS636Sx25SMTRLFS
Connections:
- net GND: now also D1.1 (K), D2.1 (K), D3.1 (K), SW2.2
- net P3.2: now reaches U1.10 (P3.3)
- net P3.2: now also R3.1
- net P3.4: now reaches U1.11 (P3.4)
- net P3.4: now also R4.1
- net P1.7: now reaches U1.5 (P1.7)
- net P1.7: now also SW2.1
- net P1.1: now reaches U1.9 (P1.1)
- net P1.1: now also R2.1
- new net: D2.2 (A), R3.2
- new net: D3.2 (A), R4.2
- new net: D1.2 (A), R2.2
Other:
- moved on the sheet: C1, C2, J1, R1, SW1, U1
