File: badUSB/badUSB.kicad_pcb (KiCad board)
At the start: 2 copper layers, 16.4 x 54.9 mm, 13 parts, among them J1 USB_A, SW1 SW_Push, SW2 SW_Push, U1 CH552G

Commit message: pcb work almost done
Parts:
- added Screw: M3, MountingHole:MountingHole_3.2mm_M3, F.Cu at (160.9, 62.8)
- moved D3 8.69 mm to (155.1, 62.8), turned to -90 degrees
- moved D1 8.51 mm to (167.0, 62.8), turned to -90 degrees
- moved R1 8.42 mm to (168.4, 87.9)
- moved SW1 1.70 mm to (161.5, 76.5)
- moved D2 1.53 mm to (157.2, 81.8)
- moved SW2 1.45 mm to (161.5, 69.8)
- moved R2 0.85 mm to (156.1, 93.7)
- moved R3 0.85 mm to (157.8, 93.7)
- moved R4 0.85 mm to (159.6, 93.7)
Routing:
- net Net-(D3-A): track 58.6 -> 39.2 mm
- net +3V3: track 16.0 -> 6.87 mm
- net Net-(R1-Pad2): track 5.27 -> 13.0 mm, vias 2 -> 0
- net /D+: track 49.7 -> 42.1 mm, vias 2 -> 0
- net Net-(D1-A): track 34.7 -> 41.9 mm
- net Net-(D2-A): track 20.8 -> 19.0 mm
- net /D-: track 15.9 -> 14.7 mm
- net /P3.2: track 3.67 -> 2.82 mm
- net /P1.1: track 3.85 -> 3.00 mm
- net /P3.4: track 3.48 -> 2.63 mm
- net GND: track 0.00 -> 0.12 mm, vias 0 -> 5
- added copper zone on B.Cu, net GND
- added copper zone on F.Cu, net GND
Other:
- board size 16.4 x 54.9 mm -> 16.5 x 53.5 mm
- board text added: "D2"
